Commit message: Refatora módulo de simulação no Gazebo

File: simulation/gazebo/carrinho.urdf (robot description, URDF)
Before this commit: robot carrinho, 4 links, 3 joints
Links:
- removed link indicador_frente
- removed link roda_dir
- removed link roda_esq
- added link front_indicator; visual box size=0.02 0.02 0.02
- added link left_wheel, mass 0.05; collision cylinder length=0.025 radius=0.0325; visual cylinder length=0.025 radius=0.0325
- added link right_wheel, mass 0.05; collision cylinder length=0.025 radius=0.0325; visual cylinder length=0.025 radius=0.0325
Joints:
- removed joint joint_dir
- removed joint joint_esq
- removed joint joint_indicador
- added joint front_indicator_joint: type fixed, parent base_link, child front_indicator, origin xyz=0.065 0 0.0825
- added joint left_wheel_joint: type fixed, parent base_link, child left_wheel, origin xyz=0 0.0675 0.0325
- added joint right_wheel_joint: type fixed, parent base_link, child right_wheel, origin xyz=0 -0.0675 0.0325
